File: v6/1tm32.sch (EAGLE design)
At the start: 44 parts, among them IC1 STM32L412RBT6, J1 DST310S_32.768KHZ, J2 10118192-0001LF, U2 LD39050PU33R, Y1 8MHz

Commit message: made changes to traces
Connections:
- net I2C2_SCL: now also JP1.11, JP1.3, JP1.7, JP4.3; no longer JP1.1, JP1.5, JP1.9, JP4.1
- net I2C2_SDA: now also JP1.1, JP1.5, JP1.9, JP4.1; no longer JP1.11, JP1.3, JP1.7, JP4.3
Changed lines of the file:
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@@
 </segment>
 <segment>
-<pinref part="JP4" gate="A" pin="1"/>
-<wire x1="53.34" y1="-53.34" x2="33.02" y2="-53.34" width="0.1524" layer="91"/>
-<label x="33.02" y="-53.34" size="1.778" layer="95"/>
+<pinref part="JP1" gate="A" pin="3"/>
+<wire x1="45.72" y1="-68.58" x2="25.4" y2="-68.58" width="0.1524" layer="91"/>
+<label x="25.4" y="-68.58" size="1.778" layer="95"/>
+</segment>
+<segment>
+<pinref part="JP1" gate="A" pin="7"/>
+<wire x1="45.72" y1="-73.66" x2="25.4" y2="-73.66" width="0.1524" layer="91"/>
+<label x="25.4" y="-73.66" size="1.778" layer="95"/>
+</segment>
+<segment>
+<pinref part="JP1" gate="A" pin="11"/>
+<wire x1="45.72" y1="-78.74" x2="25.4" y2="-78.74" width="0.1524" layer="91"/>
+<label x="25.4" y="-78.74" size="1.778" layer="95"/>
+</segment>
+<segment>
+<pinref part="JP4" gate="A" pin="3"/>
+<wire x1="53.34" y1="-55.88" x2="33.02" y2="-55.88" width="0.1524" layer="91"/>
+<label x="33.02" y="-55.88" size="1.778" layer="95"/>
+</segment>
+</net>
+<net name="I2C2_SDA" class="0">
+<segment>
+<pinref part="IC1" gate="G$1" pin="PB14"/>
+<wire x1="68.58" y1="15.24" x2="93.98" y2="15.24" width="0.1524" layer="91"/>
+<label x="76.2" y="15.24" size="1.778" layer="95"/>
 </segment>
 <segment>
@@
 <label x="25.4" y="-76.2" size="1.778" layer="95"/>
 </segment>
-</net>
-<net name="I2C2_SDA" class="0">
 <segment>
-<pinref part="IC1" gate="G$1" pin="PB14"/>
-<wire x1="68.58" y1="15.24" x2="93.98" y2="15.24" width="0.1524" layer="91"/>
-<label x="76.2" y="15.24" size="1.778" layer="95"/>
-</segment>
-<segment>
-<pinref part="JP4" gate="A" pin="3"/>
-<wire x1="53.34" y1="-55.88" x2="33.02" y2="-55.88" width="0.1524" layer="91"/>
-<label x="33.02" y="-55.88" size="1.778" layer="95"/>
-</segment>
-<segment>
-<pinref part="JP1" gate="A" pin="3"/>
-<wire x1="45.72" y1="-68.58" x2="25.4" y2="-68.58" width="0.1524" layer="91"/>
-<label x="25.4" y="-68.58" size="1.778" layer="95"/>
-</segment>
-<segment>
-<pinref part="JP1" gate="A" pin="7"/>
-<wire x1="45.72" y1="-73.66" x2="25.4" y2="-73.66" width="0.1524" layer="91"/>
-<label x="25.4" y="-73.66" size="1.778" layer="95"/>
-</segment>
-<segment>
-<pinref part="JP1" gate="A" pin="11"/>
-<wire x1="45.72" y1="-78.74" x2="25.4" y2="-78.74" width="0.1524" layer="91"/>
-<label x="25.4" y="-78.74" size="1.778" layer="95"/>
+<pinref part="JP4" gate="A" pin="1"/>
+<wire x1="53.34" y1="-53.34" x2="33.02" y2="-53.34" width="0.1524" layer="91"/>
+<label x="33.02" y="-53.34" size="1.778" layer="95"/>
 </segment>
 </net>
