File: v6/1tm32.brd (EAGLE design)
At the start: 50.8 x 50.8 mm, 44 parts, among them IC1 STM32L412RBT6, J1 DST310S_32.768KHZ, J2 10118192-0001LF, U2 LD39050PU33R, Y1 8MHz

Commit message: made changes to traces
Connections:
- net I2C2_SCL: now also JP1.11, JP1.3, JP1.7, JP4.3; no longer JP1.1, JP1.5, JP1.9, JP4.1
- net I2C2_SDA: now also JP1.1, JP1.5, JP1.9, JP4.1; no longer JP1.11, JP1.3, JP1.7, JP4.3
Routing:
- net I2C2_SDA: track 42.7 -> 47.3 mm
- net I2C2_SCL: track 43.5 -> 41.5 mm, vias 6 -> 0
- net TIM1_CH3: track 23.4 -> 23.8 mm, vias 2 -> 0

Commit message: Add files via upload
Routing:
- net USART3_TX: track 14.1 -> 15.2 mm
Changed lines of the file:
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@@
 <text x="7.62" y="36.7284" size="0.6096" layer="21" rot="R270">T1_4</text>
 <text x="8.1534" y="26.797" size="0.6096" layer="21" rot="R90">T1_2</text>
-<text x="10.8458" y="1.7526" size="0.6096" layer="21">PB13</text>
-<text x="13.589" y="1.6764" size="0.6096" layer="21">PB14</text>
+<text x="13.4874" y="1.7272" size="0.6096" layer="21">PB13</text>
+<text x="10.922" y="1.7018" size="0.6096" layer="21">PB14</text>
 <text x="11.0998" y="7.7216" size="0.6096" layer="21">PC0</text>
 <text x="13.843" y="7.6962" size="0.6096" layer="21">PC1</text>
@@
 <contactref element="IC1" pad="51"/>
 <contactref element="JP3" pad="3"/>
-<wire x1="28.943" y1="31.482" x2="28.943" y2="34.0992" width="0.2032" layer="1"/>
-<wire x1="28.943" y1="34.0992" x2="29.464" y2="34.6202" width="0.2032" layer="1"/>
+<wire x1="28.943" y1="31.482" x2="27.6344" y2="32.7906" width="0.2032" layer="1"/>
+<wire x1="27.6344" y1="32.7906" x2="29.464" y2="34.6202" width="0.2032" layer="1"/>
 <via x="29.464" y="34.6202" extent="1-16" drill="0.35"/>
 <wire x1="29.464" y1="34.6202" x2="29.464" y2="42.037" width="0.2032" layer="16"/>
